Commit message: urdf

File: assets/bookmark1_template.urdf (robot description, URDF)
Before this commit: robot template_name, 1 links, 0 joints
Links:
- link baseLink: geometry collision mesh filename=bookmark1.obj scale=1.0 1.0 1.0; visual mesh filename=bookmark1.obj scale=1.0 1.0 1.0

File: assets/bookmark2_template.urdf (robot description, URDF)
Before this commit: robot template_name, 1 links, 0 joints
Links:
- link baseLink: geometry collision mesh filename=bookmark2.obj scale=1.0 1.0 1.0; visual mesh filename=bookmark2.obj scale=1.0 1.0 1.0

File: assets/knife_template.urdf (robot description, URDF)
Before this commit: robot template_name, 1 links, 0 joints
Links:
- link baseLink: geometry collision mesh filename=knife.obj scale=1.0 1.0 1.0; visual mesh filename=knife.obj scale=1.0 1.0 1.0
